Commit message: Fix ar4 gripper.

File: ar4_gazebo_sim/urdf/includes/gazebo.xacro (robot description, xacro)
@@ -1,4 +1,5 @@
 <?xml version="1.0"?>
 <robot name="ar4" xmlns:xacro="http://www.ros.org/wiki/xacro">
+    <xacro:include filename="$(find ar4_gazebo)/urdf/ar_gripper.ros2_control.xacro" />
     <gazebo reference="base_link">
         <selfCollide>true</selfCollide>
@@ -22,4 +23,10 @@
         <selfCollide>true</selfCollide>
     </gazebo>
+    <gazebo reference="gripper_jaw1_joint">
+        <selfCollide>true</selfCollide>
+    </gazebo>
+    <gazebo reference="gripper_jaw2_joint">
+        <selfCollide>true</selfCollide>
+    </gazebo>
     <gazebo>
         <plugin filename="libign_ros2_control-system.so"

File: ar4_gazebo_sim/urdf/includes/ros2_control.xacro (robot description, xacro)
@@ -35,4 +35,14 @@
       <state_interface name="velocity" />
     </joint>
+    <joint name="gripper_jaw1_joint">
+      <command_interface name="position"/>
+      <state_interface name="position"/>
+      <state_interface name="velocity"/>
+    </joint>
+    <joint name="gripper_jaw2_joint">
+      <command_interface name="position"/>
+      <state_interface name="position"/>
+      <state_interface name="velocity"/>
+    </joint>
   </ros2_control>
 </robot>
