Commit message: Fix some issues.

File: ar4_gazebo/urdf/ar4.ros2_control.xacro (robot description, xacro)
@@ -35,9 +35,9 @@
         <state_interface name="velocity"/>
       </joint>
-      <!-- <joint name="gripper_jaw1_joint">
+      <joint name="gripper_jaw1_joint">
         <command_interface name="position"/>
         <state_interface name="position"/>
         <state_interface name="velocity"/>
-      </joint> -->
+      </joint>
     </ros2_control>
     <gazebo>
