Commit message: Fix ar4 gripper.

File: ar4_description/urdf/include/ar_gripper_macro.xacro (robot description, xacro)
@@ -72,5 +72,5 @@
       <child link="gripper_jaw1_link"/>
       <axis xyz="1 0 0"/>
-      <limit lower="-0.014" upper="0" effort="-1" velocity="1.0"/>
+      <limit lower="-0.014" upper="0" effort="100" velocity="1.0"/>
     </joint>
     <joint name="gripper_jaw2_joint" type="prismatic">
@@ -79,5 +79,5 @@
       <child link="gripper_jaw2_link"/>
       <axis xyz="1 0 0"/>
-      <limit lower="-0.014" upper="0" effort="-1" velocity="1.0"/>
+      <limit lower="-0.014" upper="0" effort="100" velocity="1.0"/>
       <mimic joint="gripper_jaw1_joint" multiplier="1" offset="0"/>
     </joint>

File: ar4_gazebo/urdf/ar4.ros2_control.xacro (robot description, xacro)
@@ -35,4 +35,9 @@
         <state_interface name="velocity"/>
       </joint>
+      <!-- <joint name="gripper_jaw1_joint">
+        <command_interface name="position"/>
+        <state_interface name="position"/>
+        <state_interface name="velocity"/>
+      </joint> -->
     </ros2_control>
     <gazebo>

File: ar4_gazebo/urdf/ar4_gazebo.urdf.xacro (robot description, xacro)
@@ -3,4 +3,5 @@
   <xacro:include filename="$(find ar4_description)/urdf/ar4.urdf.xacro" />.
   <xacro:include filename="$(find ar4_gazebo)/urdf/ar4.ros2_control.xacro" />
+  <xacro:include filename="$(find ar4_gazebo)/urdf/ar_gripper.ros2_control.xacro" />
   <link name="world" />
   <joint name="joint_world" type="fixed">
@@ -30,3 +31,9 @@
       <selfCollide>true</selfCollide>
   </gazebo>
+  <gazebo reference="gripper_jaw1_joint">
+      <selfCollide>true</selfCollide>
+  </gazebo>
+  <gazebo reference="gripper_jaw2_joint">
+      <selfCollide>true</selfCollide>
+  </gazebo>
 </robot>

Commit message: Add gripper changes

File: ar4_description/urdf/include/ar_gripper_macro.xacro (robot description, xacro)
@@ -49,4 +49,5 @@
     <link name="gripper_jaw2_link">
       <visual>
+        <!-- <origin rpy="0 3.14159265359 0" xyz="0 0 0" /> -->
         <geometry>
           <mesh filename="file://$(find ar4_description)/meshes/ar4_gripper/gripper_jaw2_link.stl" />
@@ -57,4 +58,5 @@
       </visual>
       <collision>
+        <!-- <origin rpy="0 3.14159265359 0" xyz="0 0 0" /> -->
         <geometry>
           <mesh filename="file://$(find ar4_description)/meshes/ar4_gripper/gripper_jaw2_link.stl" />

File: ar4_gazebo/urdf/ar4_gazebo.urdf.xacro (robot description, xacro)
@@ -3,5 +3,5 @@
   <xacro:include filename="$(find ar4_description)/urdf/ar4.urdf.xacro" />.
   <xacro:include filename="$(find ar4_gazebo)/urdf/ar4.ros2_control.xacro" />
-  <xacro:include filename="$(find ar4_gazebo)/urdf/ar_gripper.ros2_control.xacro" />
+  <!-- <xacro:include filename="$(find ar4_gazebo)/urdf/ar_gripper.ros2_control.xacro" /> -->
   <link name="world" />
   <joint name="joint_world" type="fixed">

File: ar4_gazebo/urdf/ar_gripper.ros2_control.xacro (robot description, xacro)
@@ -1,13 +1,7 @@
 <?xml version="1.0"?>
 <robot xmlns:xacro="http://www.ros.org/wiki/xacro">
-  <xacro:macro name="ar_gripper_ros2_control" params="
-    name
-    plugin_name
-    serial_port
-  ">
-    <ros2_control name="${name}" type="system">
+    <ros2_control name="GripperGazeboSystem" type="system">
       <hardware>
-        <plugin>${plugin_name}</plugin>
-        <param name="serial_port">${serial_port}</param>
+        <plugin>ign_ros2_control/IgnitionSystem</plugin>
       </hardware>
       <joint name="gripper_jaw1_joint">
@@ -31,4 +25,3 @@
       </joint>
     </ros2_control>
-  </xacro:macro>
 </robot>

Commit message: Gripper working correctly, I need to fix issue about gripper finger on move it.

File: ar4_description/urdf/include/ar_gripper_macro.xacro (robot description, xacro)
@@ -76,5 +76,5 @@
       <limit lower="-0.014" upper="0" effort="100" velocity="1.0"/>
     </joint>
-    <joint name="gripper_jaw2_joint" type="prismatic">
+    <joint name="gripper_jaw2_joint_mimic" type="prismatic">
       <origin xyz="0.0 -0.036 0" rpy="0.0 ${-pi} 0.0"/>
       <parent link="gripper_base_link"/>

File: ar4_gazebo/urdf/ar4.ros2_control.xacro (robot description, xacro)
@@ -35,9 +35,14 @@
         <state_interface name="velocity"/>
       </joint>
-      <joint name="gripper_jaw1_joint">
+      <!-- <joint name="gripper_jaw1_joint">
         <command_interface name="position"/>
         <state_interface name="position"/>
         <state_interface name="velocity"/>
       </joint>
+      <joint name="gripper_jaw2_joint">
+        <command_interface name="position"/>
+        <state_interface name="position"/>
+        <state_interface name="velocity"/>
+      </joint> -->
     </ros2_control>
     <gazebo>

File: ar4_gazebo/urdf/ar4_gazebo.urdf.xacro (robot description, xacro)
@@ -3,5 +3,5 @@
   <xacro:include filename="$(find ar4_description)/urdf/ar4.urdf.xacro" />.
   <xacro:include filename="$(find ar4_gazebo)/urdf/ar4.ros2_control.xacro" />
-  <!-- <xacro:include filename="$(find ar4_gazebo)/urdf/ar_gripper.ros2_control.xacro" /> -->
+  <xacro:include filename="$(find ar4_gazebo)/urdf/ar_gripper.ros2_control.xacro" />
   <link name="world" />
   <joint name="joint_world" type="fixed">
@@ -31,9 +31,9 @@
       <selfCollide>true</selfCollide>
   </gazebo>
-  <gazebo reference="gripper_jaw1_joint">
+  <!-- <gazebo reference="gripper_jaw1_joint">
       <selfCollide>true</selfCollide>
   </gazebo>
   <gazebo reference="gripper_jaw2_joint">
       <selfCollide>true</selfCollide>
-  </gazebo>
+  </gazebo> -->
 </robot>

File: ar4_gazebo_sim/urdf/includes/ar_gripper.ros2_control.xacro (robot description, xacro)
@@ -14,5 +14,5 @@
         </state_interface>
       </joint>
-      <joint name="gripper_jaw2_joint">
+      <joint name="gripper_jaw2_joint_mimic">
         <param name="mimic">gripper_jaw1_joint</param>
         <param name="multiplier">1</param>
