Commit message: added gripper files
checkpoint

added gripper to robot description

Signed-off-by: SantiagoLM <sanlopz93@gmail.com>

File: ar4_description/urdf/include/common_macros.urdf.xacro (robot description, xacro)
@@ -20,5 +20,5 @@
                      ${visual['origin']['dz']}"/>
         <geometry>
-          <mesh filename="package://ar4_description/meshes/${link_name}.STL"/>
+          <mesh filename="package://ar4_description/meshes/ar4/${link_name}.STL"/>
         </geometry>
         <material name="">
@@ -34,5 +34,5 @@
                      ${collision['origin']['dz']}"/>
         <geometry>
-          <mesh filename="package://ar4_description/meshes/${link_name}.STL"/>
+          <mesh filename="package://ar4_description/meshes/ar4/${link_name}.STL"/>
         </geometry>
       </collision>

Commit message: Clean up gazebo launch files
Signed-off-by: Francisco Rossi <frossi@ekumenlabs.com>

File: ar4_description/urdf/include/common_macros.urdf.xacro (robot description, xacro)
@@ -20,5 +20,5 @@
                      ${visual['origin']['dz']}"/>
         <geometry>
-          <mesh filename="package://ar4_description/meshes/${link_name}.STL"/>
+           <mesh filename="file://$(find ar4_description)/meshes/${link_name}.STL"/>
         </geometry>
         <material name="">
@@ -34,5 +34,5 @@
                      ${collision['origin']['dz']}"/>
         <geometry>
-          <mesh filename="package://ar4_description/meshes/${link_name}.STL"/>
+          <mesh filename="file://$(find ar4_description)/meshes/${link_name}.STL"/>
         </geometry>
       </collision>

File: ar4_gazebo/urdf/ar4_gazebo.urdf.xacro (robot description, xacro)
@@ -1,10 +1,6 @@
 <?xml version="1.0"?>
 <robot name="ar4" xmlns:xacro="http://www.ros.org/wiki/xacro">
-  <!-- Defines the Lewis component tag. -->
-  <xacro:arg name="use_gazebo_ros_control" default="true"/>
   <xacro:include filename="$(find ar4_description)/urdf/ar4.urdf.xacro" />.
-  <xacro:if value="$(arg use_gazebo_ros_control)">
-    <xacro:include filename="$(find ar4_gazebo)/urdf/ar4.ros2_control.xacro" />
-  </xacro:if>
+  <xacro:include filename="$(find ar4_gazebo)/urdf/ar4.ros2_control.xacro" />
   <link name="world" />
   <joint name="joint_world" type="fixed">

Commit message: updates to use gripper with isaac and moveit

File: ar4_description/urdf/include/common_macros.urdf.xacro (robot description, xacro)
@@ -65,6 +65,6 @@
       <parent link="gripper_base_link"/>
       <child link="finger_link_${number}"/>
-      <axis xyz="1 0 0"/>
-      <limit lower="-0.014" upper="0" effort="100" velocity="1.0"/>
+      <axis xyz="-1 0 0"/>
+      <limit upper="0.014" lower="0.0" effort="100" velocity="1.0"/>
       <xacro:if value="${mimic}">
         <mimic joint="finger_joint_1" multiplier="1" offset="0"/>

File: ar4_isaac/urdf/ar4.ros2_control.xacro (robot description, xacro)
@@ -37,4 +37,9 @@
         <state_interface name="velocity"/>
       </joint>
+        <joint name="finger_joint_1">
+          <command_interface name="position"/>
+          <state_interface name="position"/>
+          <state_interface name="velocity"/>
+      </joint>
     </ros2_control>
 </robot>

File: ar4_isaac/urdf/ar4_isaac.urdf.xacro (robot description, xacro)
@@ -3,4 +3,5 @@
   <xacro:include filename="$(find ar4_description)/urdf/ar4.urdf.xacro" />.
   <xacro:include filename="$(find ar4_isaac)/urdf/ar4.ros2_control.xacro" />
+  <!--<xacro:include filename="$(find ar4_isaac)/urdf/ar_gripper.ros2_control.xacro" />-->
   <link name="world" />
   <joint name="joint_world" type="fixed">

Commit message: Fix gripper base rotation

File: ar4_description/urdf/include/common_macros.urdf.xacro (robot description, xacro)
@@ -43,5 +43,5 @@
   <xacro:macro name="gripper_base" params="parent *origin inertial visual collision">
     <joint name="gripper_base_joint" type="fixed">
-      <origin xyz="0.0 0.0 0.0" rpy="${-pi/2} 0.0 ${pi}"/>
+      <origin xyz="0.0 0.0 0.0" rpy="${-pi/2} 0.0 0"/>
       <parent link="${parent}"/>
       <child link="gripper_base_link"/>
