Commit message: Fix robot inertias
Signed-off-by: Steven Desvars <steven.desvars@ekumenlabs.com>

File: ar4_description/urdf/ar4.urdf.xacro (robot description, xacro)
@@ -24,5 +24,5 @@
     <child link="link_1"/>
     <axis xyz="0 0 1"/>
-    <limit lower="${-170.0 / 180.0 * pi}" upper="${170.0 / 180.0 * pi}" effort="0" velocity="0.5"/>
+    <limit lower="${-170.0 / 180.0 * pi}" upper="${170.0 / 180.0 * pi}" effort="100" velocity="0.5"/>
   </joint>
   <xacro:link link_name="link_2"
@@ -37,5 +37,5 @@
     <child link="link_2"/>
     <axis xyz="0 0 1"/>
-    <limit lower="${-42.0 / 180.0 * pi}" upper="${90.0 / 180.0 * pi}" effort="0.5" velocity="0.5"/>
+    <limit lower="${-42.0 / 180.0 * pi}" upper="${90.0 / 180.0 * pi}" effort="100" velocity="0.5"/>
   </joint>
   <xacro:link link_name="link_3"
@@ -50,5 +50,5 @@
     <child link="link_3"/>
     <axis xyz="0 0 1"/>
-    <limit lower="${-89.0 / 180.0 * pi}" upper="${52.0 / 180.0 * pi}" effort="0" velocity="0.5"/>
+    <limit lower="${-89.0 / 180.0 * pi}" upper="${52.0 / 180.0 * pi}" effort="100" velocity="0.5"/>
   </joint>
   <xacro:link link_name="link_4"
@@ -63,5 +63,5 @@
     <child link="link_4"/>
     <axis xyz="0 0 1"/>
-    <limit lower="${-1 * robot_parameters['j4_limit']}" upper="${robot_parameters['j4_limit']}" effort="0" velocity="0.5"/>
+    <limit lower="${-1 * robot_parameters['j4_limit']}" upper="${robot_parameters['j4_limit']}" effort="100" velocity="0.5"/>
   </joint>
   <xacro:link link_name="link_5"
@@ -76,5 +76,5 @@
     <child link="link_5"/>
     <axis xyz="0 0 1"/>
-    <limit lower="${-105.0 / 180.0 * pi}" upper="${105.0 / 180.0 * pi}" effort="0" velocity="1.0"/>
+    <limit lower="${-105.0 / 180.0 * pi}" upper="${105.0 / 180.0 * pi}" effort="100" velocity="1.0"/>
   </joint>
   <xacro:link link_name="link_6"
@@ -89,5 +89,5 @@
     <child link="link_6"/>
     <axis xyz="0 0 1"/>
-    <limit lower="${-1.0 * robot_parameters['j6_limit']}" upper="${robot_parameters['j6_limit']}" effort="0" velocity="1.0"/>
+    <limit lower="${-1.0 * robot_parameters['j6_limit']}" upper="${robot_parameters['j6_limit']}" effort="100" velocity="1.0"/>
   </joint>
 </robot>

File: ar4_description/urdf/include/common_macros.urdf.xacro (robot description, xacro)
@@ -1,22 +1,15 @@
 <?xml version="1.0"?>
 <robot xmlns:xacro="http://www.ros.org/wiki/xacro">
+<!-- ===================== Arm link xacro ================================== -->
   <xacro:macro name="link" params="link_name *origin inertial visual collision">
     <link name="${link_name}">
       <xacro:insert_block name="origin"/>
-      <inertial>
-        <origin rpy="${inertial['origin']['dr']}
-                     ${inertial['origin']['dp']}
-                     ${inertial['origin']['dY']}"
-                xyz="${inertial['origin']['dx']}
-                     ${inertial['origin']['dy']}
-                     ${inertial['origin']['dz']}"/>
-        <mass value="${inertial['mass']}"/>
-        <inertia ixx="${inertial['inertia']['ixx']}"
-                 ixy="${inertial['inertia']['ixy']}"
-                 ixz="${inertial['inertia']['ixz']}"
-                 iyy="${inertial['inertia']['iyy']}"
-                 iyz="${inertial['inertia']['iyz']}"
-                 izz="${inertial['inertia']['izz']}"/>
-      </inertial>
+      <xacro:box_inertia m="${inertial['mass']}"
+                         x="${inertial['size']['dx']}"
+                         y="${inertial['size']['dy']}"
+                         z="${inertial['size']['dz']}"
+                         o_xyz="${inertial['origin']['dx']} ${inertial['origin']['dy']} ${inertial['origin']['dz']}"
+                         o_rpy="${inertial['origin']['dr']} ${inertial['origin']['dp']} ${inertial['origin']['dY']}">
+      </xacro:box_inertia>
       <visual>
         <origin rpy="${visual['origin']['dr']}
@@ -46,3 +39,21 @@
     </link>
   </xacro:macro>
+<!-- ===================== Box inertia xacro ==================================
+  params:
+  - m [float]: link mass;
+  - x [float]: link dimension on the X-axis;
+  - y [float]: link dimension on the Y-axis;
+  - z [float]: link dimension on the Z-axis;
+  - o_xyz [string]: position offset
+  - o_rpy [string]: rotation offset
+-->
+ <xacro:macro name="box_inertia" params="m x y z o_xyz:='0.0 0.0 0.0' o_rpy:='0.0 0.0 0.0'">
+    <inertial>
+      <mass value="${m}"/>
+      <inertia ixx="${m / 12.0 * (y*y + z*z)}" ixy="0.0" ixz="0.0"
+               iyy="${m / 12.0 * (x*x + z*z)}" iyz="0.0"
+               izz="${m / 12.0 * (x*x + y*y)}"/>
+      <origin xyz="${o_xyz}" rpy="${o_rpy}" />
+    </inertial>
+  </xacro:macro>
 </robot>

Commit message: added gripper files
checkpoint

added gripper to robot description

Signed-off-by: SantiagoLM <sanlopz93@gmail.com>

File: ar4_description/urdf/ar4.urdf.xacro (robot description, xacro)
@@ -2,4 +2,5 @@
 <robot name="ar4" xmlns:xacro="http://www.ros.org/wiki/xacro">
   <xacro:property name="package_name" value="ar4_description"/>
+  <xacro:arg name="include_gripper" default="true"/>
   <xacro:include filename="$(find ${package_name})/urdf/include/common_macros.urdf.xacro" />
   <xacro:property name="robot_properties_yaml_dir" value="$(find ${package_name})/config/link_properties.yaml" />
@@ -91,3 +92,7 @@
     <limit lower="${-1.0 * robot_parameters['j6_limit']}" upper="${robot_parameters['j6_limit']}" effort="100" velocity="1.0"/>
   </joint>
+  <xacro:if value="$(arg include_gripper)">
+    <xacro:include filename="$(find ${package_name})/urdf/include/ar_gripper_macro.xacro" />
+    <xacro:ar_gripper parent="link_6" />
+  </xacro:if>
 </robot>

File: ar4_description/urdf/include/common_macros.urdf.xacro (robot description, xacro)
@@ -20,5 +20,5 @@
                      ${visual['origin']['dz']}"/>
         <geometry>
-           <mesh filename="file://$(find ar4_description)/meshes/${link_name}.STL"/>
+           <mesh filename="file://$(find ar4_description)/meshes/ar4/${link_name}.STL"/>
         </geometry>
         <material name="">
@@ -34,5 +34,5 @@
                      ${collision['origin']['dz']}"/>
         <geometry>
-          <mesh filename="file://$(find ar4_description)/meshes/${link_name}.STL"/>
+          <mesh filename="file://$(find ar4_description)/meshes/ar4/${link_name}.STL"/>
         </geometry>
       </collision>

Commit message: added gripper files
checkpoint

added gripper to robot description

Signed-off-by: SantiagoLM <sanlopz93@gmail.com>

File: ar4_description/urdf/ar4.urdf.xacro (robot description, xacro)
@@ -2,4 +2,5 @@
 <robot name="ar4" xmlns:xacro="http://www.ros.org/wiki/xacro">
   <xacro:property name="package_name" value="ar4_description"/>
+  <xacro:arg name="include_gripper" default="true"/>
   <xacro:include filename="$(find ${package_name})/urdf/include/common_macros.urdf.xacro" />
   <xacro:property name="robot_properties_yaml_dir" value="$(find ${package_name})/config/link_properties.yaml" />
@@ -105,3 +106,7 @@
     <limit lower="${-1.0 * robot_parameters['j6_limit']}" upper="${robot_parameters['j6_limit']}" effort="100" velocity="1.0"/>
   </joint>
+  <xacro:if value="$(arg include_gripper)">
+    <xacro:include filename="$(find ${package_name})/urdf/include/ar_gripper_macro.xacro" />
+    <xacro:ar_gripper parent="link_6" />
+  </xacro:if>
 </robot>

File: ar4_description/urdf/include/common_macros.urdf.xacro (robot description, xacro)
@@ -25,5 +25,5 @@
               xyz="${visual['origin']['dx']} ${visual['origin']['dy']} ${visual['origin']['dz']}"/>
       <geometry>
-         <mesh filename="file://$(find ar4_description)/meshes/${mesh}.stl"/>
+         <mesh filename="file://$(find ar4_description)/meshes/ar4/${mesh}.stl"/>
       </geometry>
       <material name="${material}"/>
@@ -33,5 +33,5 @@
               xyz="${collision['origin']['dx']} ${collision['origin']['dy']} ${collision['origin']['dz']}"/>
       <geometry>
-        <mesh filename="file://$(find ar4_description)/meshes/${mesh}.stl"/>
+        <mesh filename="file://$(find ar4_description)/meshes/ar4/${mesh}.stl"/>
       </geometry>
     </collision>

Commit message: Update AR4 model
Signed-off-by: Francisco Rossi <frossi@ekumenlabs.com>

File: ar4_description/urdf/ar4.urdf.xacro (robot description, xacro)
@@ -10,5 +10,7 @@
               inertial="${robot_properties['base_link']['inertial']}"
               visual="${robot_properties['base_link']['visual']}"
-              collision="${robot_properties['base_link']['collision']}">
+              collision="${robot_properties['base_link']['collision']}"
+              mesh_files="${['base_link', 'base_link_bottom', 'base_link_motor']}"
+              mesh_materials="${['grey', 'blue', 'black']}">
               <origin xyz="0 0 0" rpy="0 0 0" />
   </xacro:link>
@@ -16,5 +18,7 @@
               inertial="${robot_properties['link_1']['inertial']}"
               visual="${robot_properties['link_1']['visual']}"
-              collision="${robot_properties['link_1']['collision']}">
+              collision="${robot_properties['link_1']['collision']}"
+              mesh_files="${['link_1', 'link_1_motor']}"
+              mesh_materials="${['grey', 'black']}">
     <origin xyz="0 0 0" rpy="0 0 0" />
   </xacro:link>
@@ -29,5 +33,7 @@
               inertial="${robot_properties['link_2']['inertial']}"
               visual="${robot_properties['link_2']['visual']}"
-              collision="${robot_properties['link_2']['collision']}">
+              collision="${robot_properties['link_2']['collision']}"
+              mesh_files="${['link_2', 'link_2_motor', 'link_2_cover', 'link_2_cover_logo']}"
+              mesh_materials="${['grey', 'black', 'white', 'blue']}">
     <origin xyz="0 0 0" rpy="0 0 0" />
   </xacro:link>
@@ -42,5 +48,7 @@
               inertial="${robot_properties['link_3']['inertial']}"
               visual="${robot_properties['link_3']['visual']}"
-              collision="${robot_properties['link_3']['collision']}">
+              collision="${robot_properties['link_3']['collision']}"
+              mesh_files="${['link_3', 'link_3_motor', 'link_3_misc']}"
+              mesh_materials="${['grey', 'black', 'black']}">
     <origin xyz="0 0 0" rpy="0 0 0" />
   </xacro:link>
@@ -55,5 +63,7 @@
               inertial="${robot_properties['link_4']['inertial']}"
               visual="${robot_properties['link_4']['visual']}"
-              collision="${robot_properties['link_4']['collision']}">
+              collision="${robot_properties['link_4']['collision']}"
+              mesh_files="${['link_4', 'link_4_motor']}"
+              mesh_materials="${['grey', 'black']}">
     <origin xyz="0 0 0" rpy="0 0 0" />
   </xacro:link>
@@ -68,5 +78,7 @@
               inertial="${robot_properties['link_5']['inertial']}"
               visual="${robot_properties['link_5']['visual']}"
-              collision="${robot_properties['link_5']['collision']}">
+              collision="${robot_properties['link_5']['collision']}"
+              mesh_files="${['link_5', 'link_5_motor']}"
+              mesh_materials="${['grey', 'black']}">
     <origin xyz="0 0 0" rpy="0 0 0" />
   </xacro:link>
@@ -81,5 +93,7 @@
               inertial="${robot_properties['link_6']['inertial']}"
               visual="${robot_properties['link_6']['visual']}"
-              collision="${robot_properties['link_6']['collision']}">
+              collision="${robot_properties['link_6']['collision']}"
+              mesh_files="${['link_6']}"
+              mesh_materials="${['grey']}">
     <origin xyz="0 0 0" rpy="0 0 0" />
   </xacro:link>

File: ar4_description/urdf/include/common_macros.urdf.xacro (robot description, xacro)
@@ -2,41 +2,46 @@
 <robot xmlns:xacro="http://www.ros.org/wiki/xacro">
 <!-- ===================== Arm link xacro ================================== -->
-  <xacro:macro name="link" params="link_name *origin inertial visual collision">
-    <link name="${link_name}">
-      <xacro:insert_block name="origin"/>
-      <xacro:box_inertia m="${inertial['mass']}"
-                         x="${inertial['size']['dx']}"
-                         y="${inertial['size']['dy']}"
-                         z="${inertial['size']['dz']}"
-                         o_xyz="${inertial['origin']['dx']} ${inertial['origin']['dy']} ${inertial['origin']['dz']}"
-                         o_rpy="${inertial['origin']['dr']} ${inertial['origin']['dp']} ${inertial['origin']['dY']}">
-      </xacro:box_inertia>
-      <visual>
-        <origin rpy="${visual['origin']['dr']}
-                     ${visual['origin']['dp']}
-                     ${visual['origin']['dY']}"
-                xyz="${visual['origin']['dx']}
-                     ${visual['origin']['dy']}
-                     ${visual['origin']['dz']}"/>
-        <geometry>
-           <mesh filename="file://$(find ar4_description)/meshes/${link_name}.STL"/>
-        </geometry>
-        <material name="">
-          <color rgba="1 1 0 1"/>
-        </material>
-      </visual>
-      <collision>
-        <origin rpy="${collision['origin']['dr']}
-                     ${collision['origin']['dp']}
-                     ${collision['origin']['dY']}"
-                xyz="${collision['origin']['dx']}
-                     ${collision['origin']['dy']}
-                     ${collision['origin']['dz']}"/>
-        <geometry>
-          <mesh filename="file://$(find ar4_description)/meshes/${link_name}.STL"/>
-        </geometry>
-      </collision>
-    </link>
-  </xacro:macro>
+<xacro:include filename="$(find ${package_name})/urdf/include/materials.xacro" />
+<xacro:macro name="link" params="link_name *origin inertial visual collision mesh_files:=^ mesh_materials:=^">
+  <link name="${link_name}">
+    <xacro:insert_block name="origin"/>
+    <xacro:box_inertia m="${inertial['mass']}"
+                       x="${inertial['size']['dx']}"
+                       y="${inertial['size']['dy']}"
+                       z="${inertial['size']['dz']}"
+                       o_xyz="${inertial['origin']['dx']} ${inertial['origin']['dy']} ${inertial['origin']['dz']}"
+                       o_rpy="${inertial['origin']['dr']} ${inertial['origin']['dp']} ${inertial['origin']['dY']}">
+    </xacro:box_inertia>
+    <!-- Recursively process each mesh -->
+    <xacro:property name="mesh_list" value="${mesh_files}" />
+    <xacro:property name="mesh_materials_list" value="${mesh_materials}" />
+    <xacro:mesh_loop mesh_list="${mesh_list}" mesh_materials="${mesh_materials_list}" visual="${visual}" collision="${collision}" />
+  </link>
+</xacro:macro>
+<!-- Recursive macro to iterate over meshes -->
+<xacro:macro name="mesh_loop" params="mesh_list:=^ mesh_materials:=^ visual collision">
+  <xacro:if value="${mesh_list}">
+    <!-- Pop the first mesh from the list -->
+    <xacro:property name="mesh_file" value="${mesh_list.pop(0)}"/>
+    <xacro:property name="mesh_material" value="${mesh_materials.pop(0)}"/>
+    <visual>
+      <origin rpy="${visual['origin']['dr']} ${visual['origin']['dp']} ${visual['origin']['dY']}"
+              xyz="${visual['origin']['dx']} ${visual['origin']['dy']} ${visual['origin']['dz']}"/>
+      <geometry>
+         <mesh filename="file://$(find ar4_description)/new_meshes/${mesh_file}.stl"/>
+      </geometry>
+      <material name="${mesh_material}"/>
+    </visual>
+    <collision>
+      <origin rpy="${collision['origin']['dr']} ${collision['origin']['dp']} ${collision['origin']['dY']}"
+              xyz="${collision['origin']['dx']} ${collision['origin']['dy']} ${collision['origin']['dz']}"/>
+      <geometry>
+        <mesh filename="file://$(find ar4_description)/new_meshes/${mesh_file}.stl"/>
+      </geometry>
+    </collision>
+    <!-- Recursive call to process the remaining list -->
+    <xacro:mesh_loop mesh_list="${mesh_list}" visual="${visual}" collision="${collision}" />
+  </xacro:if>
+</xacro:macro>
 <!-- ===================== Box inertia xacro ================================== -->
 <!-- params -->
