Commit message: Update AR4 model
Signed-off-by: Francisco Rossi <frossi@ekumenlabs.com>

File: ar4_description/urdf/ar4.urdf.xacro (robot description, xacro)
@@ -10,5 +10,7 @@
               inertial="${robot_properties['base_link']['inertial']}"
               visual="${robot_properties['base_link']['visual']}"
-              collision="${robot_properties['base_link']['collision']}">
+              collision="${robot_properties['base_link']['collision']}"
+              meshes="${['base_link', 'base_link_bottom', 'base_link_motor']}"
+              materials="${['grey', 'blue', 'black']}">
               <origin xyz="0 0 0" rpy="0 0 0" />
   </xacro:link>
@@ -16,5 +18,7 @@
               inertial="${robot_properties['link_1']['inertial']}"
               visual="${robot_properties['link_1']['visual']}"
-              collision="${robot_properties['link_1']['collision']}">
+              collision="${robot_properties['link_1']['collision']}"
+              meshes="${['link_1', 'link_1_motor']}"
+              materials="${['grey', 'black']}">
     <origin xyz="0 0 0" rpy="0 0 0" />
   </xacro:link>
@@ -29,5 +33,7 @@
               inertial="${robot_properties['link_2']['inertial']}"
               visual="${robot_properties['link_2']['visual']}"
-              collision="${robot_properties['link_2']['collision']}">
+              collision="${robot_properties['link_2']['collision']}"
+              meshes="${['link_2', 'link_2_motor', 'link_2_cover', 'link_2_cover_logo']}"
+              materials="${['grey', 'black', 'white', 'blue']}">
     <origin xyz="0 0 0" rpy="0 0 0" />
   </xacro:link>
@@ -42,5 +48,7 @@
               inertial="${robot_properties['link_3']['inertial']}"
               visual="${robot_properties['link_3']['visual']}"
-              collision="${robot_properties['link_3']['collision']}">
+              collision="${robot_properties['link_3']['collision']}"
+              meshes="${['link_3', 'link_3_motor', 'link_3_misc']}"
+              materials="${['grey', 'black', 'black']}">
     <origin xyz="0 0 0" rpy="0 0 0" />
   </xacro:link>
@@ -55,5 +63,7 @@
               inertial="${robot_properties['link_4']['inertial']}"
               visual="${robot_properties['link_4']['visual']}"
-              collision="${robot_properties['link_4']['collision']}">
+              collision="${robot_properties['link_4']['collision']}"
+              meshes="${['link_4', 'link_4_motor']}"
+              materials="${['grey', 'black']}">
     <origin xyz="0 0 0" rpy="0 0 0" />
   </xacro:link>
@@ -68,5 +78,7 @@
               inertial="${robot_properties['link_5']['inertial']}"
               visual="${robot_properties['link_5']['visual']}"
-              collision="${robot_properties['link_5']['collision']}">
+              collision="${robot_properties['link_5']['collision']}"
+              meshes="${['link_5', 'link_5_motor']}"
+              materials="${['grey', 'black']}">
     <origin xyz="0 0 0" rpy="0 0 0" />
   </xacro:link>
@@ -81,5 +93,7 @@
               inertial="${robot_properties['link_6']['inertial']}"
               visual="${robot_properties['link_6']['visual']}"
-              collision="${robot_properties['link_6']['collision']}">
+              collision="${robot_properties['link_6']['collision']}"
+              meshes="${['link_6']}"
+              materials="${['grey']}">
     <origin xyz="0 0 0" rpy="0 0 0" />
   </xacro:link>

File: ar4_description/urdf/include/common_macros.urdf.xacro (robot description, xacro)
@@ -2,41 +2,42 @@
 <robot xmlns:xacro="http://www.ros.org/wiki/xacro">
 <!-- ===================== Arm link xacro ================================== -->
-  <xacro:macro name="link" params="link_name *origin inertial visual collision">
-    <link name="${link_name}">
-      <xacro:insert_block name="origin"/>
-      <xacro:box_inertia m="${inertial['mass']}"
-                         x="${inertial['size']['dx']}"
-                         y="${inertial['size']['dy']}"
-                         z="${inertial['size']['dz']}"
-                         o_xyz="${inertial['origin']['dx']} ${inertial['origin']['dy']} ${inertial['origin']['dz']}"
-                         o_rpy="${inertial['origin']['dr']} ${inertial['origin']['dp']} ${inertial['origin']['dY']}">
-      </xacro:box_inertia>
-      <visual>
-        <origin rpy="${visual['origin']['dr']}
-                     ${visual['origin']['dp']}
-                     ${visual['origin']['dY']}"
-                xyz="${visual['origin']['dx']}
-                     ${visual['origin']['dy']}
-                     ${visual['origin']['dz']}"/>
-        <geometry>
-           <mesh filename="file://$(find ar4_description)/meshes/${link_name}.STL"/>
-        </geometry>
-        <material name="">
-          <color rgba="1 1 0 1"/>
-        </material>
-      </visual>
-      <collision>
-        <origin rpy="${collision['origin']['dr']}
-                     ${collision['origin']['dp']}
-                     ${collision['origin']['dY']}"
-                xyz="${collision['origin']['dx']}
-                     ${collision['origin']['dy']}
-                     ${collision['origin']['dz']}"/>
-        <geometry>
-          <mesh filename="file://$(find ar4_description)/meshes/${link_name}.STL"/>
-        </geometry>
-      </collision>
-    </link>
-  </xacro:macro>
+<xacro:include filename="$(find ${package_name})/urdf/include/materials.xacro" />
+<xacro:macro name="link" params="link_name *origin inertial visual collision meshes:=^ materials:=^">
+  <link name="${link_name}">
+    <xacro:insert_block name="origin"/>
+    <xacro:box_inertia m="${inertial['mass']}"
+                       x="${inertial['size']['dx']}"
+                       y="${inertial['size']['dy']}"
+                       z="${inertial['size']['dz']}"
+                       o_xyz="${inertial['origin']['dx']} ${inertial['origin']['dy']} ${inertial['origin']['dz']}"
+                       o_rpy="${inertial['origin']['dr']} ${inertial['origin']['dp']} ${inertial['origin']['dY']}">
+    </xacro:box_inertia>
+    <xacro:mesh_loop meshes="${meshes}" materials="${materials}" visual="${visual}" collision="${collision}" />
+  </link>
+</xacro:macro>
+<!-- Recursive macro to iterate over meshes -->
+<xacro:macro name="mesh_loop" params="meshes:=^ materials:=^ visual collision">
+  <xacro:if value="${meshes}">
+    <xacro:property name="mesh" value="${meshes.pop(0)}"/>
+    <xacro:property name="material" value="${materials.pop(0)}"/>
+    <visual>
+      <origin rpy="${visual['origin']['dr']} ${visual['origin']['dp']} ${visual['origin']['dY']}"
+              xyz="${visual['origin']['dx']} ${visual['origin']['dy']} ${visual['origin']['dz']}"/>
+      <geometry>
+         <mesh filename="file://$(find ar4_description)/meshes/${mesh}.stl"/>
+      </geometry>
+      <material name="${material}"/>
+    </visual>
+    <collision>
+      <origin rpy="${collision['origin']['dr']} ${collision['origin']['dp']} ${collision['origin']['dY']}"
+              xyz="${collision['origin']['dx']} ${collision['origin']['dy']} ${collision['origin']['dz']}"/>
+      <geometry>
+        <mesh filename="file://$(find ar4_description)/meshes/${mesh}.stl"/>
+      </geometry>
+    </collision>
+    <!-- Recursive call to process the remaining list -->
+    <xacro:mesh_loop meshes="${meshes}" materials="${materials}" visual="${visual}" collision="${collision}" />
+  </xacro:if>
+</xacro:macro>
 <!-- ===================== Box inertia xacro ================================== -->
 <!-- params -->

Commit message: Add gripper to xacro
Signed-off-by: Steven Desvars <steven.desvars@ekumenlabs.com>

File: ar4_description/urdf/ar4.urdf.xacro (robot description, xacro)
@@ -105,3 +105,25 @@
     <limit lower="${-1.0 * robot_parameters['j6_limit']}" upper="${robot_parameters['j6_limit']}" effort="100" velocity="1.0"/>
   </joint>
+  <xacro:gripper_base parent="link_6"
+                      inertial="${robot_properties['gripper_base']['inertial']}"
+                      visual="${robot_properties['gripper_base']['visual']}"
+                      collision="${robot_properties['gripper_base']['collision']}">
+    <origin xyz="0 0 0" rpy="0 0 0" />
+  </xacro:gripper_base>
+  <xacro:finger number="1"
+                pitch_rotation="0.0"
+                mimic="false"
+                inertial="${robot_properties['finger']['inertial']}"
+                visual="${robot_properties['finger']['visual']}"
+                collision="${robot_properties['finger']['collision']}">
+    <origin xyz="0 0 0" rpy="0 0 0" />
+  </xacro:finger>
+  <xacro:finger number="2"
+                pitch_rotation="${-pi}"
+                mimic="true"
+                inertial="${robot_properties['finger']['inertial']}"
+                visual="${robot_properties['finger']['visual']}"
+                collision="${robot_properties['finger']['collision']}">
+    <origin xyz="0 0 0" rpy="0 0 0" />
+  </xacro:finger>
 </robot>

File: ar4_description/urdf/include/common_macros.urdf.xacro (robot description, xacro)
@@ -40,4 +40,47 @@
   </xacro:if>
 </xacro:macro>
+<!-- ===================== Gripper base xacro ================================== -->
+  <xacro:macro name="gripper_base" params="parent *origin inertial visual collision">
+    <joint name="gripper_base_joint" type="fixed">
+      <origin xyz="0.0 0.0 0.0" rpy="${-pi/2} 0.0 ${pi}"/>
+      <parent link="${parent}"/>
+      <child link="gripper_base_link"/>
+    </joint>
+    <link name="gripper_base_link">
+      <xacro:insert_block name="origin"/>
+      <xacro:box_inertia m="${inertial['mass']}"
+                         x="${inertial['size']['dx']}"
+                         y="${inertial['size']['dy']}"
+                         z="${inertial['size']['dz']}"
+                         o_xyz="${inertial['origin']['dx']} ${inertial['origin']['dy']} ${inertial['origin']['dz']}"
+                         o_rpy="${inertial['origin']['dr']} ${inertial['origin']['dp']} ${inertial['origin']['dY']}">
+      </xacro:box_inertia>
+      <xacro:mesh_loop meshes="${['gripper_base']}" materials="${['grey']}" visual="${visual}" collision="${collision}" />
+    </link>
+  </xacro:macro>
+<!-- ===================== Gripper finger ================================== -->
+  <xacro:macro name="finger" params="number pitch_rotation mimic *origin inertial visual collision">
+    <joint name="finger_joint${number}" type="prismatic">
+      <origin xyz="0.0 -0.036 0" rpy="0.0 ${pitch_rotation} 0.0"/>
+      <parent link="gripper_base_link"/>
+      <child link="finger${number}"/>
+      <axis xyz="1 0 0"/>
+      <limit lower="-0.014" upper="0" effort="100" velocity="1.0"/>
+      <xacro:if value="${mimic == 'true'}">
+        <mimic joint="finger_joint1" multiplier="1" offset="0"/>
+      </xacro:if>
+    </joint>
+    <link name="finger${number}">
+      <xacro:insert_block name="origin"/>
+      <xacro:box_inertia m="${inertial['mass']}"
+                         x="${inertial['size']['dx']}"
+                         y="${inertial['size']['dy']}"
+                         z="${inertial['size']['dz']}"
+                         o_xyz="${inertial['origin']['dx']} ${inertial['origin']['dy']} ${inertial['origin']['dz']}"
+                         o_rpy="${inertial['origin']['dr']} ${inertial['origin']['dp']} ${inertial['origin']['dY']}">
+      </xacro:box_inertia>
+      <xacro:mesh_loop meshes="${['gripper_finger']}" materials="${['black']}" visual="${visual}" collision="${collision}" />
+    </link>
+  </xacro:macro>
 <!-- ===================== Box inertia xacro ================================== -->
 <!-- params -->

Commit message: Add gripper to xacro
Signed-off-by: Steven Desvars <steven.desvars@ekumenlabs.com>

File: ar4_description/urdf/ar4.urdf.xacro (robot description, xacro)
@@ -114,7 +114,25 @@
   </joint>
   <link name="dummy"/>
-  <xacro:if value="$(arg include_gripper)">
-    <xacro:include filename="$(find ${package_name})/urdf/include/ar_gripper_macro.xacro" />
-    <xacro:ar_gripper parent="link_6" />
-  </xacro:if>
+  <xacro:gripper_base parent="link_6"
+                      inertial="${robot_properties['gripper_base']['inertial']}"
+                      visual="${robot_properties['gripper_base']['visual']}"
+                      collision="${robot_properties['gripper_base']['collision']}">
+    <origin xyz="0 0 0" rpy="0 0 0" />
+  </xacro:gripper_base>
+  <xacro:finger number="1"
+                pitch_rotation="0.0"
+                mimic="false"
+                inertial="${robot_properties['finger']['inertial']}"
+                visual="${robot_properties['finger']['visual']}"
+                collision="${robot_properties['finger']['collision']}">
+    <origin xyz="0 0 0" rpy="0 0 0" />
+  </xacro:finger>
+  <xacro:finger number="2"
+                pitch_rotation="${-pi}"
+                mimic="true"
+                inertial="${robot_properties['finger']['inertial']}"
+                visual="${robot_properties['finger']['visual']}"
+                collision="${robot_properties['finger']['collision']}">
+    <origin xyz="0 0 0" rpy="0 0 0" />
+  </xacro:finger>
 </robot>

File: ar4_description/urdf/include/common_macros.urdf.xacro (robot description, xacro)
@@ -40,4 +40,47 @@
   </xacro:if>
 </xacro:macro>
+<!-- ===================== Gripper base xacro ================================== -->
+  <xacro:macro name="gripper_base" params="parent *origin inertial visual collision">
+    <joint name="gripper_base_joint" type="fixed">
+      <origin xyz="0.0 0.0 0.0" rpy="${-pi/2} 0.0 ${pi}"/>
+      <parent link="${parent}"/>
+      <child link="gripper_base_link"/>
+    </joint>
+    <link name="gripper_base_link">
+      <xacro:insert_block name="origin"/>
+      <xacro:box_inertia m="${inertial['mass']}"
+                         x="${inertial['size']['dx']}"
+                         y="${inertial['size']['dy']}"
+                         z="${inertial['size']['dz']}"
+                         o_xyz="${inertial['origin']['dx']} ${inertial['origin']['dy']} ${inertial['origin']['dz']}"
+                         o_rpy="${inertial['origin']['dr']} ${inertial['origin']['dp']} ${inertial['origin']['dY']}">
+      </xacro:box_inertia>
+      <xacro:mesh_loop meshes="${['gripper_base']}" materials="${['grey']}" visual="${visual}" collision="${collision}" />
+    </link>
+  </xacro:macro>
+<!-- ===================== Gripper finger ================================== -->
+  <xacro:macro name="finger" params="number pitch_rotation mimic *origin inertial visual collision">
+    <joint name="finger_joint${number}" type="prismatic">
+      <origin xyz="0.0 -0.036 0" rpy="0.0 ${pitch_rotation} 0.0"/>
+      <parent link="gripper_base_link"/>
+      <child link="finger${number}"/>
+      <axis xyz="1 0 0"/>
+      <limit lower="-0.014" upper="0" effort="100" velocity="1.0"/>
+      <xacro:if value="${mimic == 'true'}">
+        <mimic joint="finger_joint1" multiplier="1" offset="0"/>
+      </xacro:if>
+    </joint>
+    <link name="finger${number}">
+      <xacro:insert_block name="origin"/>
+      <xacro:box_inertia m="${inertial['mass']}"
+                         x="${inertial['size']['dx']}"
+                         y="${inertial['size']['dy']}"
+                         z="${inertial['size']['dz']}"
+                         o_xyz="${inertial['origin']['dx']} ${inertial['origin']['dy']} ${inertial['origin']['dz']}"
+                         o_rpy="${inertial['origin']['dr']} ${inertial['origin']['dp']} ${inertial['origin']['dY']}">
+      </xacro:box_inertia>
+      <xacro:mesh_loop meshes="${['gripper_finger']}" materials="${['black']}" visual="${visual}" collision="${collision}" />
+    </link>
+  </xacro:macro>
 <!-- ===================== Box inertia xacro ================================== -->
 <!-- params -->

Commit message: Fix rebase and rviz error with mimic joint.

File: ar4_description/urdf/ar4.urdf.xacro (robot description, xacro)
@@ -106,4 +106,12 @@
     <limit lower="${-1.0 * robot_parameters['j6_limit']}" upper="${robot_parameters['j6_limit']}" effort="100" velocity="1.0"/>
   </joint>
+  <!-- Dummy joint to remove the  "Joint '*_mimic' not found in model 'ar4'" error-->
+  <!-- See https://github.com/ros-controls/gazebo_ros2_control/issues/173 -->
+  <joint name="gripper_jaw2_joint_mimic" type="fixed">
+    <parent link="base_link" />
+    <child link="dummy" />
+    <origin xyz="0 0 0" rpy="0 0 0" />
+  </joint>
+  <link name="dummy"/>
   <xacro:if value="$(arg include_gripper)">
     <xacro:include filename="$(find ${package_name})/urdf/include/ar_gripper_macro.xacro" />

File: ar4_description/urdf/include/ar_gripper_macro.xacro (robot description, xacro)
@@ -76,5 +76,5 @@
       <limit lower="-0.014" upper="0" effort="100" velocity="1.0"/>
     </joint>
-    <joint name="gripper_jaw2_joint_mimic" type="prismatic">
+    <joint name="gripper_jaw2_joint" type="prismatic">
       <origin xyz="0.0 -0.036 0" rpy="0.0 ${-pi} 0.0"/>
       <parent link="gripper_base_link"/>

File: ar4_gazebo_sim/urdf/includes/ar_gripper.ros2_control.xacro (robot description, xacro)
@@ -14,5 +14,5 @@
         </state_interface>
       </joint>
-      <joint name="gripper_jaw2_joint_mimic">
+      <joint name="gripper_jaw2_joint">
         <param name="mimic">gripper_jaw1_joint</param>
         <param name="multiplier">1</param>

File: ar4_gazebo_sim/urdf/includes/gazebo.xacro (robot description, xacro)
@@ -1,5 +1,5 @@
 <?xml version="1.0"?>
 <robot name="ar4" xmlns:xacro="http://www.ros.org/wiki/xacro">
-    <xacro:include filename="$(find ar4_gazebo)/urdf/ar_gripper.ros2_control.xacro" />
+    <xacro:include filename="$(find ar4_gazebo_sim)/urdf/includes/ar_gripper.ros2_control.xacro" />
     <gazebo reference="base_link">
         <selfCollide>true</selfCollide>

File: ar4_gazebo_sim/urdf/includes/ros2_control.xacro (robot description, xacro)
@@ -35,14 +35,4 @@
       <state_interface name="velocity" />
     </joint>
-    <joint name="gripper_jaw1_joint">
-      <command_interface name="position"/>
-      <state_interface name="position"/>
-      <state_interface name="velocity"/>
-    </joint>
-    <joint name="gripper_jaw2_joint">
-      <command_interface name="position"/>
-      <state_interface name="position"/>
-      <state_interface name="velocity"/>
-    </joint>
   </ros2_control>
 </robot>
