Commit message: Working to add Steven gripper.

File: ar4_description/urdf/ar4.urdf.xacro (robot description, xacro)
@@ -108,5 +108,5 @@
   <!-- Dummy joint to remove the  "Joint '*_mimic' not found in model 'ar4'" error-->
   <!-- See https://github.com/ros-controls/gazebo_ros2_control/issues/173 -->
-  <joint name="gripper_jaw2_joint_mimic" type="fixed">
+  <joint name="finger_joint_2_mimic" type="fixed">
     <parent link="base_link" />
     <child link="dummy" />

File: ar4_description/urdf/include/common_macros.urdf.xacro (robot description, xacro)
@@ -25,5 +25,5 @@
               xyz="${visual['origin']['dx']} ${visual['origin']['dy']} ${visual['origin']['dz']}"/>
       <geometry>
-         <mesh filename="file://$(find ar4_description)/meshes/ar4/${mesh}.stl"/>
+         <mesh filename="file://$(find ar4_description)/meshes/${mesh}.stl"/>
       </geometry>
       <material name="${material}"/>
@@ -33,5 +33,5 @@
               xyz="${collision['origin']['dx']} ${collision['origin']['dy']} ${collision['origin']['dz']}"/>
       <geometry>
-        <mesh filename="file://$(find ar4_description)/meshes/ar4/${mesh}.stl"/>
+        <mesh filename="file://$(find ar4_description)/meshes/${mesh}.stl"/>
       </geometry>
     </collision>
@@ -61,15 +61,15 @@
 <!-- ===================== Gripper finger ================================== -->
   <xacro:macro name="finger" params="number pitch_rotation mimic *origin inertial visual collision">
-    <joint name="finger_joint${number}" type="prismatic">
+    <joint name="finger_joint_${number}" type="prismatic">
       <origin xyz="0.0 -0.036 0" rpy="0.0 ${pitch_rotation} 0.0"/>
       <parent link="gripper_base_link"/>
-      <child link="finger${number}"/>
+      <child link="finger_link_${number}"/>
       <axis xyz="1 0 0"/>
       <limit lower="-0.014" upper="0" effort="100" velocity="1.0"/>
       <xacro:if value="${mimic == 'true'}">
-        <mimic joint="finger_joint1" multiplier="1" offset="0"/>
+        <mimic joint="finger_joint_1" multiplier="1" offset="0"/>
       </xacro:if>
     </joint>
-    <link name="finger${number}">
+    <link name="finger_link_${number}">
       <xacro:insert_block name="origin"/>
       <xacro:box_inertia m="${inertial['mass']}"

File: ar4_gazebo/urdf/ar4.ros2_control.xacro (robot description, xacro)
@@ -35,10 +35,10 @@
         <state_interface name="velocity"/>
       </joint>
-      <!-- <joint name="gripper_jaw1_joint">
+      <!-- <joint name="finger_joint_1">
         <command_interface name="position"/>
         <state_interface name="position"/>
         <state_interface name="velocity"/>
       </joint>
-      <joint name="gripper_jaw2_joint">
+      <joint name="finger_joint_2">
         <command_interface name="position"/>
         <state_interface name="position"/>

File: ar4_gazebo/urdf/ar4_gazebo.urdf.xacro (robot description, xacro)
@@ -31,8 +31,8 @@
       <selfCollide>true</selfCollide>
   </gazebo>
-  <!-- <gazebo reference="gripper_jaw1_joint">
+  <!-- <gazebo reference="finger_link_1">
       <selfCollide>true</selfCollide>
   </gazebo>
-  <gazebo reference="gripper_jaw2_joint">
+  <gazebo reference="finger_link_2">
       <selfCollide>true</selfCollide>
   </gazebo> -->

File: ar4_gazebo_sim/urdf/gz_ar4.urdf.xacro (robot description, xacro)
@@ -7,3 +7,5 @@
   <!-- ros2_control extensions -->
   <xacro:include filename="$(find ar4_gazebo_sim)/urdf/includes/ros2_control.xacro" />
+  <!-- ros2_control gripper extensions -->
+  <xacro:include filename="$(find ar4_gazebo_sim)/urdf/includes/ar_gripper.ros2_control.xacro" />
 </robot>

File: ar4_gazebo_sim/urdf/includes/ar_gripper.ros2_control.xacro (robot description, xacro)
@@ -5,5 +5,5 @@
         <plugin>ign_ros2_control/IgnitionSystem</plugin>
       </hardware>
-      <joint name="gripper_jaw1_joint">
+      <joint name="finger_joint_1">
         <command_interface name="position" />
         <state_interface name="position">
@@ -14,6 +14,6 @@
         </state_interface>
       </joint>
-      <joint name="gripper_jaw2_joint">
-        <param name="mimic">gripper_jaw1_joint</param>
+      <joint name="finger_joint_2">
+        <param name="mimic">finger_joint_1</param>
         <param name="multiplier">1</param>
         <state_interface name="position">

File: ar4_gazebo_sim/urdf/includes/gazebo.xacro (robot description, xacro)
@@ -1,5 +1,4 @@
 <?xml version="1.0"?>
 <robot name="ar4" xmlns:xacro="http://www.ros.org/wiki/xacro">
-    <xacro:include filename="$(find ar4_gazebo_sim)/urdf/includes/ar_gripper.ros2_control.xacro" />
     <gazebo reference="base_link">
         <selfCollide>true</selfCollide>
@@ -23,8 +22,8 @@
         <selfCollide>true</selfCollide>
     </gazebo>
-    <gazebo reference="gripper_jaw1_joint">
+    <gazebo reference="finger_link_1">
         <selfCollide>true</selfCollide>
     </gazebo>
-    <gazebo reference="gripper_jaw2_joint">
+    <gazebo reference="finger_link_2">
         <selfCollide>true</selfCollide>
     </gazebo>

Commit message: Adding gripper on gazebo, fix issues on moveit, fix issues on hardware. improve control implementation.
Signed-off-by: Fabricio Emder <elector102@gmail.com>

File: ar4_description/urdf/ar4.urdf.xacro (robot description, xacro)
@@ -2,5 +2,4 @@
 <robot name="ar4" xmlns:xacro="http://www.ros.org/wiki/xacro">
   <xacro:property name="package_name" value="ar4_description"/>
-  <xacro:arg name="include_gripper" default="true"/>
   <xacro:include filename="$(find ${package_name})/urdf/include/common_macros.urdf.xacro" />
   <xacro:property name="robot_properties_yaml_dir" value="$(find ${package_name})/config/link_properties.yaml" />
@@ -106,7 +105,33 @@
     <limit lower="${-1.0 * robot_parameters['j6_limit']}" upper="${robot_parameters['j6_limit']}" effort="100" velocity="1.0"/>
   </joint>
-  <xacro:if value="$(arg include_gripper)">
-    <xacro:include filename="$(find ${package_name})/urdf/include/ar_gripper_macro.xacro" />
-    <xacro:ar_gripper parent="link_6" />
-  </xacro:if>
+  <!-- Dummy joint to remove the  "Joint '*_mimic' not found in model 'ar4'" error-->
+  <!-- See https://github.com/ros-controls/gazebo_ros2_control/issues/173 -->
+  <joint name="finger_joint_2_mimic" type="fixed">
+    <parent link="base_link" />
+    <child link="dummy" />
+    <origin xyz="0 0 0" rpy="0 0 0" />
+  </joint>
+  <link name="dummy"/>
+  <xacro:gripper_base parent="link_6"
+                      inertial="${robot_properties['gripper_base']['inertial']}"
+                      visual="${robot_properties['gripper_base']['visual']}"
+                      collision="${robot_properties['gripper_base']['collision']}">
+    <origin xyz="0 0 0" rpy="0 0 0" />
+  </xacro:gripper_base>
+  <xacro:finger number="1"
+                pitch_rotation="0.0"
+                mimic="false"
+                inertial="${robot_properties['finger']['inertial']}"
+                visual="${robot_properties['finger']['visual']}"
+                collision="${robot_properties['finger']['collision']}">
+    <origin xyz="0 0 0" rpy="0 0 0" />
+  </xacro:finger>
+  <xacro:finger number="2"
+                pitch_rotation="${-pi}"
+                mimic="true"
+                inertial="${robot_properties['finger']['inertial']}"
+                visual="${robot_properties['finger']['visual']}"
+                collision="${robot_properties['finger']['collision']}">
+    <origin xyz="0 0 0" rpy="0 0 0" />
+  </xacro:finger>
 </robot>

File: ar4_description/urdf/include/common_macros.urdf.xacro (robot description, xacro)
@@ -25,5 +25,5 @@
               xyz="${visual['origin']['dx']} ${visual['origin']['dy']} ${visual['origin']['dz']}"/>
       <geometry>
-         <mesh filename="file://$(find ar4_description)/meshes/ar4/${mesh}.stl"/>
+         <mesh filename="file://$(find ar4_description)/meshes/${mesh}.stl"/>
       </geometry>
       <material name="${material}"/>
@@ -33,5 +33,5 @@
               xyz="${collision['origin']['dx']} ${collision['origin']['dy']} ${collision['origin']['dz']}"/>
       <geometry>
-        <mesh filename="file://$(find ar4_description)/meshes/ar4/${mesh}.stl"/>
+        <mesh filename="file://$(find ar4_description)/meshes/${mesh}.stl"/>
       </geometry>
     </collision>
@@ -40,4 +40,47 @@
   </xacro:if>
 </xacro:macro>
+<!-- ===================== Gripper base xacro ================================== -->
+  <xacro:macro name="gripper_base" params="parent *origin inertial visual collision">
+    <joint name="gripper_base_joint" type="fixed">
+      <origin xyz="0.0 0.0 0.0" rpy="${-pi/2} 0.0 0"/>
+      <parent link="${parent}"/>
+      <child link="gripper_base_link"/>
+    </joint>
+    <link name="gripper_base_link">
+      <xacro:insert_block name="origin"/>
+      <xacro:box_inertia m="${inertial['mass']}"
+                         x="${inertial['size']['dx']}"
+                         y="${inertial['size']['dy']}"
+                         z="${inertial['size']['dz']}"
+                         o_xyz="${inertial['origin']['dx']} ${inertial['origin']['dy']} ${inertial['origin']['dz']}"
+                         o_rpy="${inertial['origin']['dr']} ${inertial['origin']['dp']} ${inertial['origin']['dY']}">
+      </xacro:box_inertia>
+      <xacro:mesh_loop meshes="${['gripper_base']}" materials="${['grey']}" visual="${visual}" collision="${collision}" />
+    </link>
+  </xacro:macro>
+<!-- ===================== Gripper finger ================================== -->
+  <xacro:macro name="finger" params="number pitch_rotation mimic *origin inertial visual collision">
+    <joint name="finger_joint_${number}" type="prismatic">
+      <origin xyz="0.0 -0.036 0" rpy="0.0 ${pitch_rotation} 0.0"/>
+      <parent link="gripper_base_link"/>
+      <child link="finger_link_${number}"/>
+      <axis xyz="1 0 0"/>
+      <limit lower="-0.014" upper="0" effort="100" velocity="1.0"/>
+      <xacro:if value="${mimic}">
+        <mimic joint="finger_joint_1" multiplier="1" offset="0"/>
+      </xacro:if>
+    </joint>
+    <link name="finger_link_${number}">
+      <xacro:insert_block name="origin"/>
+      <xacro:box_inertia m="${inertial['mass']}"
+                         x="${inertial['size']['dx']}"
+                         y="${inertial['size']['dy']}"
+                         z="${inertial['size']['dz']}"
+                         o_xyz="${inertial['origin']['dx']} ${inertial['origin']['dy']} ${inertial['origin']['dz']}"
+                         o_rpy="${inertial['origin']['dr']} ${inertial['origin']['dp']} ${inertial['origin']['dY']}">
+      </xacro:box_inertia>
+      <xacro:mesh_loop meshes="${['gripper_finger']}" materials="${['black']}" visual="${visual}" collision="${collision}" />
+    </link>
+  </xacro:macro>
 <!-- ===================== Box inertia xacro ================================== -->
 <!-- params -->

File: ar4_gazebo_sim/urdf/gz_ar4.urdf.xacro (robot description, xacro)
@@ -7,3 +7,5 @@
   <!-- ros2_control extensions -->
   <xacro:include filename="$(find ar4_gazebo_sim)/urdf/includes/ros2_control.xacro" />
+  <!-- ros2_control gripper extensions -->
+  <xacro:include filename="$(find ar4_gazebo_sim)/urdf/includes/gripper.ros2_control.xacro" />
 </robot>

File: ar4_gazebo_sim/urdf/includes/gazebo.xacro (robot description, xacro)
@@ -22,4 +22,10 @@
         <selfCollide>true</selfCollide>
     </gazebo>
+    <gazebo reference="finger_link_1">
+        <selfCollide>true</selfCollide>
+    </gazebo>
+    <gazebo reference="finger_link_2">
+        <selfCollide>true</selfCollide>
+    </gazebo>
     <gazebo>
         <plugin filename="libign_ros2_control-system.so"

File: ar4_gazebo_sim/urdf/includes/gripper.ros2_control.xacro (robot description, xacro)
@@ -1,15 +1,9 @@
 <?xml version="1.0"?>
 <robot xmlns:xacro="http://www.ros.org/wiki/xacro">
-  <xacro:macro name="ar_gripper_ros2_control" params="
-    name
-    plugin_name
-    serial_port
-  ">
-    <ros2_control name="${name}" type="system">
+    <ros2_control name="GripperGazeboSystem" type="system">
       <hardware>
-        <plugin>${plugin_name}</plugin>
-        <param name="serial_port">${serial_port}</param>
+        <plugin>ign_ros2_control/IgnitionSystem</plugin>
       </hardware>
-      <joint name="gripper_jaw1_joint">
+      <joint name="finger_joint_1">
         <command_interface name="position" />
         <state_interface name="position">
@@ -20,6 +14,6 @@
         </state_interface>
       </joint>
-      <joint name="gripper_jaw2_joint">
-        <param name="mimic">gripper_jaw1_joint</param>
+      <joint name="finger_joint_2">
+        <param name="mimic">finger_joint_1</param>
         <param name="multiplier">1</param>
         <state_interface name="position">
@@ -31,4 +25,3 @@
       </joint>
     </ros2_control>
-  </xacro:macro>
 </robot>

Commit message: Add simplified collision meshes
Signed-off-by: Steven Desvars <steven.desvars@ekumenlabs.com>

File: ar4_description/urdf/ar4.urdf.xacro (robot description, xacro)
@@ -11,6 +11,7 @@
               visual="${robot_properties['base_link']['visual']}"
               collision="${robot_properties['base_link']['collision']}"
-              meshes="${['base_link', 'base_link_bottom', 'base_link_motor']}"
-              materials="${['grey', 'blue', 'black']}">
+              visual_meshes="${['base_link', 'base_link_bottom', 'base_link_motor']}"
+              materials="${['grey', 'blue', 'black']}"
+              collision_meshes="${['base_link_collision']}">
               <origin xyz="0 0 0" rpy="0 0 0" />
   </xacro:link>
@@ -19,6 +20,7 @@
               visual="${robot_properties['link_1']['visual']}"
               collision="${robot_properties['link_1']['collision']}"
-              meshes="${['link_1', 'link_1_motor']}"
-              materials="${['grey', 'black']}">
+              visual_meshes="${['link_1', 'link_1_motor']}"
+              materials="${['grey', 'black']}"
+              collision_meshes="${['link_1_collision']}">
     <origin xyz="0 0 0" rpy="0 0 0" />
   </xacro:link>
@@ -34,6 +36,7 @@
               visual="${robot_properties['link_2']['visual']}"
               collision="${robot_properties['link_2']['collision']}"
-              meshes="${['link_2', 'link_2_motor', 'link_2_cover', 'link_2_cover_logo']}"
-              materials="${['grey', 'black', 'white', 'blue']}">
+              visual_meshes="${['link_2', 'link_2_motor', 'link_2_cover', 'link_2_cover_logo']}"
+              materials="${['grey', 'black', 'white', 'blue']}"
+              collision_meshes="${['link_2_collision']}">
     <origin xyz="0 0 0" rpy="0 0 0" />
   </xacro:link>
@@ -49,6 +52,7 @@
               visual="${robot_properties['link_3']['visual']}"
               collision="${robot_properties['link_3']['collision']}"
-              meshes="${['link_3', 'link_3_motor', 'link_3_misc']}"
-              materials="${['grey', 'black', 'black']}">
+              visual_meshes="${['link_3', 'link_3_motor', 'link_3_misc']}"
+              materials="${['grey', 'black', 'black']}"
+              collision_meshes="${['link_3_collision']}">
     <origin xyz="0 0 0" rpy="0 0 0" />
   </xacro:link>
@@ -64,6 +68,7 @@
               visual="${robot_properties['link_4']['visual']}"
               collision="${robot_properties['link_4']['collision']}"
-              meshes="${['link_4', 'link_4_motor']}"
-              materials="${['grey', 'black']}">
+              visual_meshes="${['link_4', 'link_4_motor']}"
+              materials="${['grey', 'black']}"
+              collision_meshes="${['link_4_collision']}">
     <origin xyz="0 0 0" rpy="0 0 0" />
   </xacro:link>
@@ -79,6 +84,7 @@
               visual="${robot_properties['link_5']['visual']}"
               collision="${robot_properties['link_5']['collision']}"
-              meshes="${['link_5', 'link_5_motor']}"
-              materials="${['grey', 'black']}">
+              visual_meshes="${['link_5', 'link_5_motor']}"
+              materials="${['grey', 'black']}"
+              collision_meshes="${['link_5_collision']}">
     <origin xyz="0 0 0" rpy="0 0 0" />
   </xacro:link>
@@ -94,6 +100,7 @@
               visual="${robot_properties['link_6']['visual']}"
               collision="${robot_properties['link_6']['collision']}"
-              meshes="${['link_6']}"
-              materials="${['grey']}">
+              visual_meshes="${['link_6']}"
+              materials="${['grey']}"
+              collision_meshes="${['link_6']}">
     <origin xyz="0 0 0" rpy="0 0 0" />
   </xacro:link>

File: ar4_description/urdf/include/common_macros.urdf.xacro (robot description, xacro)
@@ -3,5 +3,5 @@
 <!-- ===================== Arm link xacro ================================== -->
 <xacro:include filename="$(find ${package_name})/urdf/include/materials.xacro" />
-<xacro:macro name="link" params="link_name *origin inertial visual collision meshes:=^ materials:=^">
+<xacro:macro name="link" params="link_name *origin inertial visual collision visual_meshes:=^ materials:=^ collision_meshes:=^">
   <link name="${link_name}">
     <xacro:insert_block name="origin"/>
@@ -13,9 +13,10 @@
                        o_rpy="${inertial['origin']['dr']} ${inertial['origin']['dp']} ${inertial['origin']['dY']}">
     </xacro:box_inertia>
-    <xacro:mesh_loop meshes="${meshes}" materials="${materials}" visual="${visual}" collision="${collision}" />
+    <xacro:mesh_loop_visuals meshes="${visual_meshes}" materials="${materials}" visual="${visual}" />
+    <xacro:mesh_loop_collisions meshes="${collision_meshes}" collision="${collision}" />
   </link>
 </xacro:macro>
-<!-- Recursive macro to iterate over meshes -->
-<xacro:macro name="mesh_loop" params="meshes:=^ materials:=^ visual collision">
+<!-- Recursive macro to iterate over visual meshes -->
+<xacro:macro name="mesh_loop_visuals" params="meshes:=^ materials:=^ visual">
   <xacro:if value="${meshes}">
     <xacro:property name="mesh" value="${meshes.pop(0)}"/>
@@ -29,4 +30,12 @@
       <material name="${material}"/>
     </visual>
+    <!-- Recursive call to process the remaining list -->
+    <xacro:mesh_loop_visuals meshes="${meshes}" materials="${materials}" visual="${visual}" />
+  </xacro:if>
+</xacro:macro>
+<!-- Recursive macro to iterate over collision meshes -->
+<xacro:macro name="mesh_loop_collisions" params="meshes:=^ collision">
+  <xacro:if value="${meshes}">
+    <xacro:property name="mesh" value="${meshes.pop(0)}"/>
     <collision>
       <origin rpy="${collision['origin']['dr']} ${collision['origin']['dp']} ${collision['origin']['dY']}"
@@ -37,5 +46,5 @@
     </collision>
     <!-- Recursive call to process the remaining list -->
-    <xacro:mesh_loop meshes="${meshes}" materials="${materials}" visual="${visual}" collision="${collision}" />
+    <xacro:mesh_loop_collisions meshes="${meshes}" collision="${collision}" />
   </xacro:if>
 </xacro:macro>
@@ -56,5 +65,6 @@
                          o_rpy="${inertial['origin']['dr']} ${inertial['origin']['dp']} ${inertial['origin']['dY']}">
       </xacro:box_inertia>
-      <xacro:mesh_loop meshes="${['gripper_base']}" materials="${['grey']}" visual="${visual}" collision="${collision}" />
+      <xacro:mesh_loop_visuals meshes="${['gripper_base']}" materials="${['grey']}" visual="${visual}" />
+      <xacro:mesh_loop_collisions meshes="${['gripper_base_collision']}" collision="${collision}" />
     </link>
   </xacro:macro>
@@ -80,5 +90,6 @@
                          o_rpy="${inertial['origin']['dr']} ${inertial['origin']['dp']} ${inertial['origin']['dY']}">
       </xacro:box_inertia>
-      <xacro:mesh_loop meshes="${['gripper_finger']}" materials="${['black']}" visual="${visual}" collision="${collision}" />
+      <xacro:mesh_loop_visuals meshes="${['gripper_finger']}" materials="${['black']}" visual="${visual}" />
+      <xacro:mesh_loop_collisions meshes="${['gripper_finger_collision']}" collision="${collision}" />
     </link>
   </xacro:macro>
