Commit message: Add gripper to MuJoCo simulation
Signed-off-by: Steven Desvars <steven.desvars@ekumenlabs.com>

File: ar4_mujoco_sim/urdf/mj_ar4.urdf (robot description, URDF)
Before this commit: robot ar4, 7 links, 6 joints
Links:
- added link dummy
- added link finger_link_1, mass 0.01; collision mesh filename=meshes/gripper_finger_collision.stl; visual mesh filename=meshes/gripper_finger.stl
- added link finger_link_2, mass 0.01; collision mesh filename=meshes/gripper_finger_collision.stl; visual mesh filename=meshes/gripper_finger.stl
- added link gripper_base_link, mass 0.08; collision mesh filename=meshes/gripper_base_collision.stl; visual mesh filename=meshes/gripper_base.stl
- link base_link: geometry collision mesh filename=meshes/base_link_collision.stl; visual mesh filename=meshes/base_link.stl
- link link_1: geometry collision mesh filename=meshes/link_1_collision.stl; visual mesh filename=meshes/link_1.stl
- link link_2: geometry collision mesh filename=meshes/link_2_collision.stl; visual mesh filename=meshes/link_2.stl
- link link_3: geometry collision mesh filename=meshes/link_3_collision.stl; visual mesh filename=meshes/link_3.stl
- link link_4: geometry collision mesh filename=meshes/link_4_collision.stl; visual mesh filename=meshes/link_4.stl
- link link_5: geometry collision mesh filename=meshes/link_5_collision.stl; visual mesh filename=meshes/link_5.stl
- link link_6: geometry collision mesh filename=meshes/link_6_collision.stl; visual mesh filename=meshes/link_6.stl
Joints:
- added joint finger_joint_1: type prismatic, parent gripper_base_link, child finger_link_1, origin xyz=0.0 -0.036 0 rpy=0.0 0.0 0.0, axis 1 0 0, limit lower=-0.014 upper=0 effort=100 velocity=1.0
- added joint finger_joint_2: type prismatic, parent gripper_base_link, child finger_link_2, origin xyz=0.0 -0.036 0 rpy=0.0 -3.141592653589793 0.0, axis 1 0 0, limit lower=-0.014 upper=0 effort=100 velocity=1.0, mimic joint=finger_joint_1 multiplier=1 offset=0
- added joint finger_joint_2_mimic: type fixed, parent base_link, child dummy, origin xyz=0 0 0 rpy=0 0 0
- added joint gripper_base_joint: type fixed, parent link_6, child gripper_base_link, origin xyz=0.0 0.0 0.0 rpy=-1.5707963267948966 0.0 0

File: ar4_mujoco_sim/xacro/mj_ar4.urdf.xacro (robot description, xacro)
@@ -7,3 +7,5 @@
   <!-- ros2_control extensions -->
   <xacro:include filename="$(find ar4_mujoco_sim)/xacro/includes/ros2_control.xacro" />
+  <!-- ros2_control gripper extensions -->
+  <xacro:include filename="$(find ar4_mujoco_sim)/xacro/includes/gripper.ros2_control.xacro" />
 </robot>

Commit message: Add gripper to MuJoCo simulation (#35)
* Add gripper to MuJoCo simulation

Signed-off-by: Steven Desvars <steven.desvars@ekumenlabs.com>

* Add equality constraint to make the grippers close

Signed-off-by: Steven Desvars <steven.desvars@ekumenlabs.com>

* Remove unnecessary meshes

Signed-off-by: Steven Desvars <steven.desvars@ekumenlabs.com>

* Add the meshes for MuJoCo

Signed-off-by: Steven Desvars <steven.desvars@ekumenlabs.com>

* Add instructions for update the model

Signed-off-by: Steven Desvars <steven.desvars@ekumenlabs.com>

* Address comments - part 1

Signed-off-by: Steven Desvars <steven.desvars@ekumenlabs.com>

---------

Signed-off-by: Steven Desvars <steven.desvars@ekumenlabs.com>

File: ar4_mujoco_sim/urdf/mj_ar4.urdf (robot description, URDF)
Before this commit: robot ar4, 7 links, 6 joints
Links:
- added link dummy
- added link finger_link_1, mass 0.01; collision mesh filename=meshes/gripper_finger_collision.stl; visual mesh filename=meshes/gripper_finger.stl
- added link finger_link_2, mass 0.01; collision mesh filename=meshes/gripper_finger_collision.stl; visual mesh filename=meshes/gripper_finger.stl
- added link gripper_base_link, mass 0.08; collision mesh filename=meshes/gripper_base_collision.stl; visual mesh filename=meshes/gripper_base.stl
- link base_link: geometry collision mesh filename=meshes/base_link_collision.stl; visual mesh filename=meshes/base_link.stl
- link link_1: geometry collision mesh filename=meshes/link_1_collision.stl; visual mesh filename=meshes/link_1.stl
- link link_2: geometry collision mesh filename=meshes/link_2_collision.stl; visual mesh filename=meshes/link_2.stl
- link link_3: geometry collision mesh filename=meshes/link_3_collision.stl; visual mesh filename=meshes/link_3.stl
- link link_4: geometry collision mesh filename=meshes/link_4_collision.stl; visual mesh filename=meshes/link_4.stl
- link link_5: geometry collision mesh filename=meshes/link_5_collision.stl; visual mesh filename=meshes/link_5.stl
- link link_6: geometry collision mesh filename=meshes/link_6_collision.stl; visual mesh filename=meshes/link_6.stl
Joints:
- added joint finger_joint_1: type prismatic, parent gripper_base_link, child finger_link_1, origin xyz=0.0 -0.036 0 rpy=0.0 0.0 0.0, axis 1 0 0, limit lower=-0.014 upper=0 effort=100 velocity=1.0
- added joint finger_joint_2: type prismatic, parent gripper_base_link, child finger_link_2, origin xyz=0.0 -0.036 0 rpy=0.0 -3.141592653589793 0.0, axis 1 0 0, limit lower=-0.014 upper=0 effort=100 velocity=1.0, mimic joint=finger_joint_1 multiplier=1 offset=0
- added joint finger_joint_2_mimic: type fixed, parent base_link, child dummy, origin xyz=0 0 0 rpy=0 0 0
- added joint gripper_base_joint: type fixed, parent link_6, child gripper_base_link, origin xyz=0.0 0.0 0.0 rpy=-1.5707963267948966 0.0 0
