Commit message: Update Isaac model to include gripper

File: ar4_isaac/urdf/ar4.ros2_control.xacro (robot description, xacro)
@@ -37,4 +37,13 @@
         <state_interface name="velocity"/>
       </joint>
+      <joint name="finger_joint_1">
+        <command_interface name="position" />
+        <state_interface name="position">
+          <param name="initial_value">0.0</param>
+        </state_interface>
+        <state_interface name="velocity">
+          <param name="initial_value">0.0</param>
+        </state_interface>
+      </joint>
     </ros2_control>
 </robot>

File: ar4_isaac/urdf/ar4_isaac.urdf.xacro (robot description, xacro)
@@ -3,4 +3,5 @@
   <xacro:include filename="$(find ar4_description)/urdf/ar4.urdf.xacro" />.
   <xacro:include filename="$(find ar4_isaac)/urdf/ar4.ros2_control.xacro" />
+  <!-- <xacro:include filename="$(find ar4_isaac)/urdf/ar_gripper.ros2_control.xacro" /> -->
   <link name="world" />
   <joint name="joint_world" type="fixed">

Commit message: Add gripper to the Isaac simulation
Signed-off-by: Steven Desvars <steven.desvars@ekumenlabs.com>

File: ar4_isaac/urdf/ar4.ros2_control.xacro (robot description, xacro)
@@ -37,4 +37,14 @@
         <state_interface name="velocity"/>
       </joint>
+      <!-- We put the gripper under the same ros2_control system because the TopicBasedSystem doesn't behave well with multiple instances-->
+      <joint name="finger_joint_1">
+        <command_interface name="position" />
+        <state_interface name="position">
+          <param name="initial_value">0.0</param>
+        </state_interface>
+        <state_interface name="velocity">
+          <param name="initial_value">0.0</param>
+        </state_interface>
+      </joint>
     </ros2_control>
 </robot>

File: ar4_isaac/urdf/ar4_isaac.urdf.xacro (robot description, xacro)
@@ -1,5 +1,7 @@
 <?xml version="1.0"?>
 <robot name="ar4" xmlns:xacro="http://www.ros.org/wiki/xacro">
+  <!-- base model -->
   <xacro:include filename="$(find ar4_description)/urdf/ar4.urdf.xacro" />.
+  <!-- ros2_control extensions -->
   <xacro:include filename="$(find ar4_isaac)/urdf/ar4.ros2_control.xacro" />
   <link name="world" />
